File: eagle/tf520.brd (EAGLE design)
At the start: 95.2 x 80 mm, 23 parts, among them IC1 MC68020, IC3 XC9536_44VQ, U1 LM1117, X1 MC68000

Commit message: Adding the Atari ST fixes Reorganizing the repos. Added jed files for rev 2 and rev 3 Published the REV 3 sources and ucf
Parts:
- added C7: 10uF, microbuilder:1206
- added IC2: 74LVC1G17DBV, 74xx-little-de:SOT23-5
- JP4: device jumper:JP1 -> SparkFun-Retired:1X02
- moved JP4 1.27 mm to (69.0, 75.4), turned to 270 degrees
Connections:
- new net CLK7M_RAW: IC2.2, X1.15
- net A0: now also IC3.32; no longer IC3.33
- net AS20: now also IC3.18; no longer IC3.19
- net AVEC: now also IC3.27; no longer IC3.28
- net BERR: now also IC3.22; no longer IC3.23
- net BG20: now also IC3.1; no longer IC3.3
- net CLK7M: now also IC2.4; no longer X1.15
- net DS20: now also IC3.16; no longer IC3.18
- net DSACK1: now also IC3.21; no longer IC3.22
- net E: now also IC3.3; no longer IC3.2
- net FC0: now also IC3.31; no longer IC3.32
- net FC1: now also IC3.23; no longer IC3.27
- net FC2: now also IC3.30; no longer IC3.31
- net GND: now also C7.2, IC2.3
- net HALT: now also IC3.20; no longer IC3.21
- net R/W20: now also IC3.19; no longer IC3.20
- net RESET: now also IC3.33
- net SIZ0: now also IC3.29; no longer IC3.30
- net SIZ1: now also IC3.28; no longer IC3.29
- net VCC: now also IC2.5
- net VCC33: now also C7.1
- net VMA: now also IC3.2; no longer IC3.1
Routing:
- net BG20: track 45.0 -> 84.2 mm, vias 2 -> 0
- net RESET: track 29.3 -> 57.9 mm
- net CLK20: track 105.3 -> 78.2 mm
- net GND: track 377.8 -> 386.3 mm
- net R/W: track 36.1 -> 28.0 mm
- net VMA: track 69.8 -> 76.5 mm
- net VCC33: track 140.0 -> 146.7 mm, vias 2 -> 4
- net CLK7M_RAW: track 0.00 -> 5.84 mm
- net D29: track 140.7 -> 135.2 mm
- net CLK7M: track 77.7 -> 72.5 mm
- net BERR: track 75.4 -> 79.4 mm
- net BGACK: track 55.6 -> 51.8 mm
- net VCC: track 341.6 -> 344.6 mm
- net A18: track 154.1 -> 156.7 mm
- net A19: track 156.5 -> 158.8 mm
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Other:
- board text added: "Revision 3"
- board text removed: "Revision 2"
